File: LP5812_dev_board.kicad_pcb (KiCad board)
At the start: 2 copper layers, 60 x 60 mm, 37 parts, among them J1 Conn_01x05, U1 LP5812ADSDR, U2 LP5812BDSDR

Commit message: Fix messed up annotations on LEDs
Connections:
- D2 pad 1: OUT2_A -> OUT1_B
- D2 pad 2: OUT1_A -> OUT0_B
- D2 pad 3: OUT0_A -> OUT3_B
- D2 pad 4: OUT3_A -> OUT2_B
- D3 pad 1: OUT3_A -> OUT2_A
- D3 pad 2: OUT2_A -> OUT1_A
- D3 pad 3: OUT1_A -> OUT0_A
- D3 pad 4: OUT0_A -> OUT3_A
- D4 pad 1: OUT0_A -> OUT2_B
- D4 pad 2: OUT3_A -> OUT1_B
- D4 pad 3: OUT2_A -> OUT0_B
- D4 pad 4: OUT1_A -> OUT3_B
- D5 pad 1: OUT1_B -> OUT3_A
- D5 pad 2: OUT0_B -> OUT2_A
- D5 pad 3: OUT3_B -> OUT1_A
- D5 pad 4: OUT2_B -> OUT0_A
- D6 pad 1: OUT2_B -> OUT3_B
- D6 pad 2: OUT1_B -> OUT2_B
- D6 pad 3: OUT0_B -> OUT1_B
- D6 pad 4: OUT3_B -> OUT0_B
- D7 pad 1: OUT0_B -> OUT0_A
- D7 pad 2: OUT3_B -> OUT3_A
- D7 pad 3: OUT2_B -> OUT2_A
- D7 pad 4: OUT1_B -> OUT1_A
- D8 pad 1: OUT3_B -> OUT0_B
- D8 pad 2: OUT2_B -> OUT3_B
- D8 pad 3: OUT1_B -> OUT2_B
- D8 pad 4: OUT0_B -> OUT1_B
- TP2 pad 1: OUT0_B -> OUT1_A
- TP3 pad 1: OUT1_A -> OUT2_A
- TP4 pad 1: OUT1_B -> OUT3_A
- TP5 pad 1: OUT2_A -> OUT0_B
- TP6 pad 1: OUT2_B -> OUT1_B
- TP7 pad 1: OUT3_A -> OUT2_B
Changed lines of the file:
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@@
 		(sheetname "Root")
 		(sheetfile "LP5812_dev_board.kicad_sch")
-		(attr smd exclude_from_bom)
+		(attr smd exclude_from_bom dnp)
 		(fp_circle
 			(center 0 0)
@@
 		(sheetname "Root")
 		(sheetfile "LP5812_dev_board.kicad_sch")
-		(attr exclude_from_pos_files)
+		(attr exclude_from_pos_files dnp)
 		(fp_circle
 			(center 0 0)
@@
 			(size 1.5 1.5)
 			(layers "F.Cu" "F.Mask")
-			(net 10 "OUT0_B")
+			(net 7 "OUT1_A")
 			(pinfunction "1")
 			(pintype "passive")
@@
 		(fp_arc
 			(start -2.655 -0.813)
-			(mid -2.6455 -0.822501)
+			(mid -2.6455 -0.822502)
 			(end -2.636 -0.813)
 			(stroke
@@
 			(size 1.1 1.4)
 			(layers "F.Cu" "F.Paste" "F.Mask")
-			(net 6 "OUT0_A")
+			(net 11 "OUT2_B")
 			(pinfunction "RK")
 			(pintype "passive")
@@
 			(size 1.1 1.4)
 			(layers "F.Cu" "F.Paste" "F.Mask")
-			(net 9 "OUT3_A")
+			(net 13 "OUT1_B")
 			(pinfunction "A")
 			(pintype "passive")
@@
 			(size 1.1 1.4)
 			(layers "F.Cu" "F.Paste" "F.Mask")
-			(net 8 "OUT2_A")
+			(net 10 "OUT0_B")
 			(pinfunction "BK")
 			(pintype "passive")
@@
 			(size 1.1 1.4)
 			(layers "F.Cu" "F.Paste" "F.Mask")
-			(net 7 "OUT1_A")
+			(net 12 "OUT3_B")
 			(pinfunction "GK")
 			(pintype "passive")
@@
 		(fp_arc
 			(start -2.655 -0.813)
-			(mid -2.6455 -0.822501)
+			(mid -2.6455 -0.822502)
 			(end -2.636 -0.813)
 			(stroke
@@
 			(size 1.1 1.4)
 			(layers "F.Cu" "F.Paste" "F.Mask")
-			(net 8 "OUT2_A")
+			(net 13 "OUT1_B")
 			(pinfunction "RK")
 			(pintype "passive")
@@
 			(size 1.1 1.4)
 			(layers "F.Cu" "F.Paste" "F.Mask")
-			(net 7 "OUT1_A")
+			(net 10 "OUT0_B")
 			(pinfunction "A")
 			(pintype "passive")
@@
 			(size 1.1 1.4)
 			(layers "F.Cu" "F.Paste" "F.Mask")
-			(net 6 "OUT0_A")
+			(net 12 "OUT3_B")
 			(pinfunction "BK")
 			(pintype "passive")
@@
 			(size 1.1 1.4)
 			(layers "F.Cu" "F.Paste" "F.Mask")
-			(net 9 "OUT3_A")
+			(net 11 "OUT2_B")
 			(pinfunction "GK")
 			(pintype "passive")
@@
 			(size 1.1 1.4)
 			(layers "F.Cu" "F.Paste" "F.Mask")
-			(net 10 "OUT0_B")
+			(net 6 "OUT0_A")
 			(pinfunction "RK")
 			(pintype "passive")
@@
 			(size 1.1 1.4)
 			(layers "F.Cu" "F.Paste" "F.Mask")
-			(net 12 "OUT3_B")
+			(net 9 "OUT3_A")
 			(pinfunction "A")
 			(pintype "passive")
@@
 			(size 1.1 1.4)
 			(layers "F.Cu" "F.Paste" "F.Mask")
-			(net 11 "OUT2_B")
+			(net 8 "OUT2_A")
 			(pinfunction "BK")
 			(pintype "passive")
@@
 			(size 1.1 1.4)
 			(layers "F.Cu" "F.Paste" "F.Mask")
-			(net 13 "OUT1_B")
+			(net 7 "OUT1_A")
 			(pinfunction "GK")
 			(pintype "passive")
@@
 			(size 1.1 1.4)
 			(layers "F.Cu" "F.Paste" "F.Mask")
-			(net 9 "OUT3_A")
+			(net 8 "OUT2_A")
 			(pinfunction "RK")
 			(pintype "passive")
@@
 			(size 1.1 1.4)
 			(layers "F.Cu" "F.Paste" "F.Mask")
-			(net 8 "OUT2_A")
+			(net 7 "OUT1_A")
 			(pinfunction "A")
 			(pintype "passive")
@@
 			(size 1.1 1.4)
 			(layers "F.Cu" "F.Paste" "F.Mask")
-			(net 7 "OUT1_A")
+			(net 6 "OUT0_A")
 			(pinfunction "BK")
 			(pintype "passive")
@@
 			(size 1.1 1.4)
 			(layers "F.Cu" "F.Paste" "F.Mask")
-			(net 6 "OUT0_A")
+			(net 9 "OUT3_A")
 			(pinfunction "GK")
 			(pintype "passive")
@@
 		(sheetname "Root")
 		(sheetfile "LP5812_dev_board.kicad_sch")
-		(attr exclude_from_pos_files)
+		(attr exclude_from_pos_files dnp)
 		(fp_circle
 			(center 0 0)
@@
 			(size 1.5 1.5)
 			(layers "F.Cu" "F.Mask")
-			(net 11 "OUT2_B")
+			(net 13 "OUT1_B")
 			(pinfunction "1")
 			(pintype "passive")
@@
 		(sheetname "Root")
 		(sheetfile "LP5812_dev_board.kicad_sch")
-		(attr exclude_from_pos_files)
+		(attr exclude_from_pos_files dnp)
 		(fp_circle
 			(center 0 0)
@@
 		(sheetname "Root")
 		(sheetfile "LP5812_dev_board.kicad_sch")
-		(attr exclude_from_pos_files)
+		(attr exclude_from_pos_files dnp)
 		(fp_circle
 			(center 0 0)
@@
 			(size 1.5 1.5)
 			(layers "F.Cu" "F.Mask")
-			(net 8 "OUT2_A")
+			(net 10 "OUT0_B")
 			(pinfunction "1")
 			(pintype "passive")
@@
 		(sheetname "Root")
 		(sheetfile "LP5812_dev_board.kicad_sch")
-		(attr exclude_from_pos_files)
+		(attr exclude_from_pos_files dnp)
 		(fp_circle
 			(center 0 0)
@@
 			(size 1.5 1.5)
 			(layers "F.Cu" "F.Mask")
-			(net 9 "OUT3_A")
+			(net 11 "OUT2_B")
 			(pinfunction "1")
 			(pintype "passive")
@@
 		)
 		(property "Value" "1u"
-			(at 0 1.43 270)
+			(at 0 1.43 -90)
 			(layer "F.Fab")
 			(effects
@@
 		)
 		(fp_text user "${REFERENCE}"
-			(at 0 0 270)
+			(at 0 0 -90)
 			(layer "F.Fab")
 			(effects
@@
 		(sheetname "Root")
 		(sheetfile "LP5812_dev_board.kicad_sch")
-		(attr exclude_from_pos_files)
+		(attr exclude_from_pos_files dnp)
 		(fp_circle
 			(center 0 0)
@@
 			(size 1.5 1.5)
 			(layers "F.Cu" "F.Mask")
-			(net 7 "OUT1_A")
+			(net 8 "OUT2_A")
 			(pinfunction "1")
 			(pintype "passive")
@@
 		(fp_arc
 			(start -2.655 -0.813)
-			(mid -2.6455 -0.822501)
+			(mid -2.6455 -0.822502)
 			(end -2.636 -0.813)
 			(stroke
@@
 			(size 1.1 1.4)
 			(layers "F.Cu" "F.Paste" "F.Mask")
-			(net 12 "OUT3_B")
+			(net 10 "OUT0_B")
 			(pinfunction "RK")
 			(pintype "passive")
@@
 			(size 1.1 1.4)
 			(layers "F.Cu" "F.Paste" "F.Mask")
-			(net 11 "OUT2_B")
+			(net 12 "OUT3_B")
 			(pinfunction "A")
 			(pintype "passive")
@@
 			(size 1.1 1.4)
 			(layers "F.Cu" "F.Paste" "F.Mask")
-			(net 13 "OUT1_B")
+			(net 11 "OUT2_B")
 			(pinfunction "BK")
 			(pintype "passive")
@@
 			(size 1.1 1.4)
 			(layers "F.Cu" "F.Paste" "F.Mask")
-			(net 10 "OUT0_B")
+			(net 13 "OUT1_B")
 			(pinfunction "GK")
 			(pintype "passive")
@@
 			(size 1.1 1.4)
 			(layers "F.Cu" "F.Paste" "F.Mask")
-			(net 13 "OUT1_B")
+			(net 9 "OUT3_A")
 			(pinfunction "RK")
 			(pintype "passive")
@@
 			(size 1.1 1.4)
 			(layers "F.Cu" "F.Paste" "F.Mask")
-			(net 10 "OUT0_B")
+			(net 8 "OUT2_A")
 			(pinfunction "A")
 			(pintype "passive")
@@
 			(size 1.1 1.4)
 			(layers "F.Cu" "F.Paste" "F.Mask")
-			(net 12 "OUT3_B")
+			(net 7 "OUT1_A")
 			(pinfunction "BK")
 			(pintype "passive")
@@
 			(size 1.1 1.4)
 			(layers "F.Cu" "F.Paste" "F.Mask")
-			(net 11 "OUT2_B")
+			(net 6 "OUT0_A")
 			(pinfunction "GK")
 			(pintype "passive")
@@
 		(sheetname "Root")
 		(sheetfile "LP5812_dev_board.kicad_sch")
-		(attr exclude_from_pos_files)
+		(attr exclude_from_pos_files dnp)
 		(fp_circle
 			(center 0 0)
@@
 		(fp_arc
 			(start -2.655 -0.813)
-			(mid -2.6455 -0.822501)
+			(mid -2.6455 -0.822502)
 			(end -2.636 -0.813)
 			(stroke
@@
 			(size 1.1 1.4)
 			(layers "F.Cu" "F.Paste" "F.Mask")
-			(net 11 "OUT2_B")
+			(net 12 "OUT3_B")
 			(pinfunction "RK")
 			(pintype "passive")
@@
 			(size 1.1 1.4)
 			(layers "F.Cu" "F.Paste" "F.Mask")
-			(net 13 "OUT1_B")
+			(net 11 "OUT2_B")
 			(pinfunction "A")
 			(pintype "passive")
@@
 			(size 1.1 1.4)
 			(layers "F.Cu" "F.Paste" "F.Mask")
-			(net 10 "OUT0_B")
+			(net 13 "OUT1_B")
 			(pinfunction "BK")
 			(pintype "passive")
@@
 			(size 1.1 1.4)
 			(layers "F.Cu" "F.Paste" "F.Mask")
-			(net 12 "OUT3_B")
+			(net 10 "OUT0_B")
 			(pinfunction "GK")
 			(pintype "passive")
@@
 		(sheetname "Root")
 		(sheetfile "LP5812_dev_board.kicad_sch")
-		(attr exclude_from_pos_files)
+		(attr exclude_from_pos_files dnp)
 		(fp_circle
 			(center 0 0)
@@
 		(sheetname "Root")
 		(sheetfile "LP5812_dev_board.kicad_sch")
-		(attr exclude_from_pos_files)
+		(attr exclude_from_pos_files dnp)
 		(fp_circle
 			(center 0 0)
@@
 			(size 1.5 1.5)
 			(layers "F.Cu" "F.Mask")
-			(net 13 "OUT1_B")
+			(net 9 "OUT3_A")
 			(pinfunction "1")
 			(pintype "passive")
@@
 		(sheetname "Root")
 		(sheetfile "LP5812_dev_board.kicad_sch")
-		(attr smd exclude_from_bom)
+		(attr smd exclude_from_bom dnp)
 		(fp_circle
 			(center 0 0)
@@
 		(sheetname "Root")
 		(sheetfile "LP5812_dev_board.kicad_sch")
-		(attr exclude_from_pos_files)
+		(attr exclude_from_pos_files dnp)
 		(fp_circle
 			(center 0 0)
@@
 		(sheetname "Root")
 		(sheetfile "LP5812_dev_board.kicad_sch")
-		(attr exclude_from_pos_files)
+		(attr exclude_from_pos_files dnp)
 		(fp_circle
 			(center 0 0)
@@
 		)
 		(property "Value" "1u"
-			(at 0 1.43 270)
+			(at 0 1.43 -90)
 			(layer "F.Fab")
 			(effects
@@
 		)
 		(fp_text user "${REFERENCE}"
-			(at 0 0 270)
+			(at 0 0 -90)
 			(layer "F.Fab")
 			(effects
@@
 		(sheetname "Root")
 		(sheetfile "LP5812_dev_board.kicad_sch")
-		(attr smd exclude_from_bom)
+		(attr smd exclude_from_bom dnp)
 		(fp_circle
 			(center 0 0)

Commit message: Route PCB and generate outputs
Parts:
- removed TP10: ~, TestPoint:TestPoint_Pad_D1.5mm
- moved TP6 31.0 mm to (126.5, 100.5)
- moved TP8 30.1 mm to (129.5, 100.5)
- moved TP3 26.5 mm to (110.5, 100.5)
- moved TP7 23.2 mm to (116.5, 100.5)
- moved TP5 22.6 mm to (113.5, 100.5)
- moved TP4 20.5 mm to (123.5, 100.5)
- moved TP1 13.6 mm to (107.5, 100.5)
- moved TP2 12.7 mm to (120.5, 100.4)
Connections:
- net Net-(J1-Pin_1) renamed /VIN
- TP2 pad 1: OUT1_A -> OUT0_B
- TP3 pad 1: OUT2_A -> OUT1_A
- TP4 pad 1: OUT3_A -> OUT1_B
- TP5 pad 1: OUT0_B -> OUT2_A
- TP6 pad 1: OUT1_B -> OUT2_B
- TP7 pad 1: OUT2_B -> OUT3_A
Routing:
- net OUT0_B: track 0.00 -> 163.0 mm
- net OUT3_B: track 0.00 -> 161.6 mm, vias 0 -> 5
- net OUT1_B: track 0.00 -> 145.1 mm, vias 0 -> 2
- net OUT2_B: track 0.00 -> 128.3 mm, vias 0 -> 2
- net OUT2_A: track 0.00 -> 123.5 mm, vias 0 -> 4
- net OUT0_A: track 0.00 -> 121.8 mm, vias 0 -> 2
- net OUT3_A: track 0.00 -> 115.1 mm, vias 0 -> 6
- net OUT1_A: track 0.00 -> 108.5 mm, vias 0 -> 6
- net VCC: track 0.00 -> 58.1 mm
- net SCL: track 0.00 -> 48.7 mm, vias 0 -> 6
- net SDA: track 0.00 -> 47.6 mm, vias 0 -> 6
- net SYNC: track 0.00 -> 24.4 mm, vias 0 -> 2
- net GND: track 0.00 -> 13.4 mm, vias 0 -> 318
- net /VIN: track 0.00 -> 7.55 mm
- added copper zone on B.Cu, net GND
- added copper zone on F.Cu, net GND
Other:
- board text added: "GND"
- board text added: "SCL"
- board text added: "SDA"
- board text added: "VIN"
- board text added: "WayWayWay"
