File: LP5812_dev_board.kicad_sch (KiCad schematic)
At the start: 34 parts, among them J1 Conn_01x05, U1 LP5812ADSDR, U2 LP5812BDSDR

Commit message: Update LEDS for better reverse bias behavior and cost
Parts:
- removed LED1, LED2, LED3, LED4, LED5, LED6, LED7, LED8: ASMB-TTF0-0A20B, ASMB-TTF0-0A20B:ASMBTTF00A20B, symbol ASMB-TTF0-0A20B:ASMB-TTF0-0A20B
- added D1, D2, D3, D4, D5, D6, D7, D8: LED_RABG, CLVBA-FKA-CAEDH8BBB7A363:CLVBAFKACAEDH8BBB7A363, symbol Device:LED_RABG
- added FID1, FID2, FID3: ~, Fiducial:Fiducial_1mm_Mask3mm, symbol Mechanical:Fiducial
Connections:
- net OUT0_A: now also D1.2 (A), D2.3 (BK), D3.4 (GK), D4.1 (RK)
- net OUT0_B: now also D5.2 (A), D6.3 (BK), D7.1 (RK), D8.4 (GK)
- net OUT1_A: now also D1.1 (RK), D2.2 (A), D3.3 (BK), D4.4 (GK)
- net OUT1_B: now also D5.1 (RK), D6.2 (A), D7.4 (GK), D8.3 (BK)
- net OUT2_A: now also D1.4 (GK), D2.1 (RK), D3.2 (A), D4.3 (BK)
- net OUT2_B: now also D5.4 (GK), D6.1 (RK), D7.3 (BK), D8.2 (A)
- net OUT3_A: now also D1.3 (BK), D2.4 (GK), D3.1 (RK), D4.2 (A)
- net OUT3_B: now also D5.3 (BK), D6.4 (GK), D7.2 (A), D8.1 (RK)
Other:
- note added: "2.7-5.5V but is practially limited by LED selection"
- note added: "Fiducial Marks"
- moved on the sheet: TP1, TP2, TP3, TP4, TP5, TP6, TP7, TP8

Commit message: Fix messed up annotations on LEDs
Parts:
- FID1, FID2, FID3, TP10, TP11, TP12: now not fitted
- TP?: renamed from TP8; now not fitted
- TP?: renamed from TP4; now not fitted
- TP?: renamed from TP6; now not fitted
- TP?: renamed from TP7; now not fitted
- TP?: renamed from TP2; now not fitted
- TP?: renamed from TP5; now not fitted
- TP?: renamed from TP3; now not fitted
- TP?: renamed from TP1; now not fitted
- renumbered D5 to D2, D2 to D3, D6 to D4, D3 to D5, D8 to D6, D4 to D7, D7 to D8
Changed lines of the file:
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@@
 		(date "2024-03-19")
 		(rev "1.0")
-		(comment 1 "All rights reserved")
-		(comment 2 "Copyright 2024 Andrew Newell")
 	)
 	(junction
@@
 		(in_bom yes)
 		(on_board yes)
-		(dnp no)
-		(property "Reference" "TP8"
+		(dnp yes)
+		(property "Reference" "TP?"
 			(at 252.476 129.54 0)
 			(effects
@@
 			(project "LP5812_dev_board"
 				(path "/a5e340e1-6f5a-42cd-9c9f-a895aae72132"
-					(reference "TP8")
+					(reference "TP?")
 					(unit 1)
 				)
@@
 		(dnp no)
 		(fields_autoplaced yes)
-		(property "Reference" "D4"
+		(property "Reference" "D7"
 			(at 260.35 59.69 0)
 			(effects
@@
 			(project "LP5812_dev_board"
 				(path "/a5e340e1-6f5a-42cd-9c9f-a895aae72132"
-					(reference "D4")
+					(reference "D7")
 					(unit 1)
 				)
@@
 		(in_bom yes)
 		(on_board yes)
-		(dnp no)
+		(dnp yes)
 		(property "Reference" "TP10"
 			(at 20.32 34.798 90)
@@
 		(in_bom yes)
 		(on_board yes)
-		(dnp no)
-		(property "Reference" "TP4"
+		(dnp yes)
+		(property "Reference" "TP?"
 			(at 252.73 98.806 0)
 			(effects
@@
 			(project "LP5812_dev_board"
 				(path "/a5e340e1-6f5a-42cd-9c9f-a895aae72132"
-					(reference "TP4")
+					(reference "TP?")
 					(unit 1)
 				)
@@
 		(in_bom no)
 		(on_board yes)
-		(dnp no)
+		(dnp yes)
 		(fields_autoplaced yes)
 		(property "Reference" "FID3"
@@
 		(in_bom no)
 		(on_board yes)
-		(dnp no)
+		(dnp yes)
 		(fields_autoplaced yes)
 		(property "Reference" "FID1"
@@
 		(in_bom yes)
 		(on_board yes)
-		(dnp no)
-		(property "Reference" "TP6"
+		(dnp yes)
+		(property "Reference" "TP?"
 			(at 212.09 129.032 0)
 			(effects
@@
 			(project "LP5812_dev_board"
 				(path "/a5e340e1-6f5a-42cd-9c9f-a895aae72132"
-					(reference "TP6")
+					(reference "TP?")
 					(unit 1)
 				)
@@
 		(in_bom yes)
 		(on_board yes)
-		(dnp no)
-		(property "Reference" "TP7"
+		(dnp yes)
+		(property "Reference" "TP?"
 			(at 252.984 64.262 0)
 			(effects
@@
 			(project "LP5812_dev_board"
 				(path "/a5e340e1-6f5a-42cd-9c9f-a895aae72132"
-					(reference "TP7")
+					(reference "TP?")
 					(unit 1)
 				)
@@
 		(in_bom yes)
 		(on_board yes)
-		(dnp no)
+		(dnp yes)
 		(property "Reference" "TP12"
 			(at 152.4 44.958 90)
@@
 		(dnp no)
 		(fields_autoplaced yes)
-		(property "Reference" "D6"
+		(property "Reference" "D4"
 			(at 260.35 93.98 0)
 			(effects
@@
 			(project "LP5812_dev_board"
 				(path "/a5e340e1-6f5a-42cd-9c9f-a895aae72132"
-					(reference "D6")
+					(reference "D4")
 					(unit 1)
 				)
@@
 		(in_bom yes)
 		(on_board yes)
-		(dnp no)
-		(property "Reference" "TP2"
+		(dnp yes)
+		(property "Reference" "TP?"
 			(at 212.09 99.06 0)
 			(effects
@@
 			(project "LP5812_dev_board"
 				(path "/a5e340e1-6f5a-42cd-9c9f-a895aae72132"
-					(reference "TP2")
+					(reference "TP?")
 					(unit 1)
 				)
@@
 		(in_bom yes)
 		(on_board yes)
-		(dnp no)
+		(dnp yes)
 		(property "Reference" "TP11"
 			(at 96.52 46.228 90)
@@
 		(in_bom yes)
 		(on_board yes)
-		(dnp no)
-		(property "Reference" "TP5"
+		(dnp yes)
+		(property "Reference" "TP?"
 			(at 212.09 64.77 0)
 			(effects
@@
 			(project "LP5812_dev_board"
 				(path "/a5e340e1-6f5a-42cd-9c9f-a895aae72132"
-					(reference "TP5")
+					(reference "TP?")
 					(unit 1)
 				)
@@
 		(dnp no)
 		(fields_autoplaced yes)
-		(property "Reference" "D5"
+		(property "Reference" "D2"
 			(at 219.71 93.98 0)
 			(effects
@@
 			(project "LP5812_dev_board"
 				(path "/a5e340e1-6f5a-42cd-9c9f-a895aae72132"
-					(reference "D5")
+					(reference "D2")
 					(unit 1)
 				)
@@
 		(dnp no)
 		(fields_autoplaced yes)
-		(property "Reference" "D3"
+		(property "Reference" "D5"
 			(at 219.71 59.69 0)
 			(effects
@@
 			(project "LP5812_dev_board"
 				(path "/a5e340e1-6f5a-42cd-9c9f-a895aae72132"
-					(reference "D3")
+					(reference "D5")
 					(unit 1)
 				)
@@
 		(dnp no)
 		(fields_autoplaced yes)
-		(property "Reference" "D2"
+		(property "Reference" "D3"
 			(at 260.35 29.21 0)
 			(effects
@@
 			(project "LP5812_dev_board"
 				(path "/a5e340e1-6f5a-42cd-9c9f-a895aae72132"
-					(reference "D2")
+					(reference "D3")
 					(unit 1)
 				)
@@
 		(in_bom yes)
 		(on_board yes)
-		(dnp no)
-		(property "Reference" "TP3"
+		(dnp yes)
+		(property "Reference" "TP?"
 			(at 252.476 34.29 0)
 			(effects
@@
 			(project "LP5812_dev_board"
 				(path "/a5e340e1-6f5a-42cd-9c9f-a895aae72132"
-					(reference "TP3")
+					(reference "TP?")
 					(unit 1)
 				)
@@
 		(dnp no)
 		(fields_autoplaced yes)
-		(property "Reference" "D8"
+		(property "Reference" "D6"
 			(at 219.71 124.46 0)
 			(effects
@@
 			(project "LP5812_dev_board"
 				(path "/a5e340e1-6f5a-42cd-9c9f-a895aae72132"
-					(reference "D8")
+					(reference "D6")
 					(unit 1)
 				)
@@
 		(in_bom yes)
 		(on_board yes)
-		(dnp no)
-		(property "Reference" "TP1"
+		(dnp yes)
+		(property "Reference" "TP?"
 			(at 212.09 34.036 0)
 			(effects
@@
 			(project "LP5812_dev_board"
 				(path "/a5e340e1-6f5a-42cd-9c9f-a895aae72132"
-					(reference "TP1")
+					(reference "TP?")
 					(unit 1)
 				)
@@
 		(in_bom no)
 		(on_board yes)
-		(dnp no)
+		(dnp yes)
 		(fields_autoplaced yes)
 		(property "Reference" "FID2"
@@
 		(dnp no)
 		(fields_autoplaced yes)
-		(property "Reference" "D7"
+		(property "Reference" "D8"
 			(at 260.35 124.46 0)
 			(effects
@@
 			(project "LP5812_dev_board"
 				(path "/a5e340e1-6f5a-42cd-9c9f-a895aae72132"
-					(reference "D7")
+					(reference "D8")
 					(unit 1)
 				)

Commit message: Route PCB and generate outputs
Parts:
- removed TP10: ~, TestPoint:TestPoint_Pad_D1.5mm, symbol Connector:TestPoint
- gave numbers to parts that had none: 8
Connections:
- net VIN: now reaches C7.1, FB1.2, J1.1 (Pin_1)
Changed lines of the file:
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@@
 	)
 	(junction
-		(at 24.13 36.83)
-		(diameter 0)
-		(color 0 0 0 0)
-	)
-	(junction
 		(at 26.67 40.64)
 		(diameter 0)
@@
 		)
 	)
+	(label "VIN"
+		(at 26.67 72.39 180)
+		(fields_autoplaced yes)
+		(effects
+			(font
+				(size 1.27 1.27)
+			)
+			(justify right bottom)
+		)
+	)
 	(global_label "OUT2_B"
 		(shape bidirectional)
@@
 		(on_board yes)
 		(dnp yes)
-		(property "Reference" "TP?"
+		(property "Reference" "TP8"
 			(at 252.476 129.54 0)
 			(effects
@@
 			(project "LP5812_dev_board"
 				(path "/a5e340e1-6f5a-42cd-9c9f-a895aae72132"
-					(reference "TP?")
+					(reference "TP8")
 					(unit 1)
 				)
@@
 	)
 	(symbol
-		(lib_id "Connector:TestPoint")
-		(at 24.13 36.83 90)
-		(unit 1)
-		(exclude_from_sim no)
-		(in_bom yes)
-		(on_board yes)
-		(dnp yes)
-		(property "Reference" "TP10"
-			(at 20.32 34.798 90)
-			(effects
-				(font
-					(size 1.27 1.27)
-				)
-			)
-		)
-		(property "Value" "~"
-			(at 20.828 34.29 90)
-			(effects
-				(font
-					(size 1.27 1.27)
-				)
-			)
-		)
-		(property "Footprint" "TestPoint:TestPoint_Pad_D1.5mm"
-			(at 24.13 31.75 0)
-			(effects
-				(font
-					(size 1.27 1.27)
-				)
-				(hide yes)
-			)
-		)
-		(property "Datasheet" "~"
-			(at 24.13 31.75 0)
-			(effects
-				(font
-					(size 1.27 1.27)
-				)
-				(hide yes)
-			)
-		)
-		(property "Description" "test point"
-			(at 24.13 36.83 0)
-			(effects
-				(font
-					(size 1.27 1.27)
-				)
-				(hide yes)
-			)
-		)
-		(property "Height" ""
-			(at 24.13 36.83 0)
-			(effects
-				(font
-					(size 1.27 1.27)
-				)
-				(hide yes)
-			)
-		)
-		(property "Manufacturer_Name" ""
-			(at 24.13 36.83 0)
-			(effects
-				(font
-					(size 1.27 1.27)
-				)
-				(hide yes)
-			)
-		)
-		(property "Manufacturer_Part_Number" ""
-			(at 24.13 36.83 0)
-			(effects
-				(font
-					(size 1.27 1.27)
-				)
-				(hide yes)
-			)
-		)
-		(property "Mouser Part Number" ""
-			(at 24.13 36.83 0)
-			(effects
-				(font
-					(size 1.27 1.27)
-				)
-				(hide yes)
-			)
-		)
-		(pin "1"
-		)
-		(instances
-			(project "LP5812_dev_board"
-				(path "/a5e340e1-6f5a-42cd-9c9f-a895aae72132"
-					(reference "TP10")
-					(unit 1)
-				)
-			)
-		)
-	)
-	(symbol
 		(lib_id "Device:C")
 		(at 35.56 66.04 90)
@@
 		(on_board yes)
 		(dnp yes)
-		(property "Reference" "TP?"
+		(property "Reference" "TP4"
 			(at 252.73 98.806 0)
 			(effects
@@
 			(project "LP5812_dev_board"
 				(path "/a5e340e1-6f5a-42cd-9c9f-a895aae72132"
-					(reference "TP?")
+					(reference "TP4")
 					(unit 1)
 				)
@@
 		(on_board yes)
 		(dnp yes)
-		(property "Reference" "TP?"
+		(property "Reference" "TP6"
 			(at 212.09 129.032 0)
 			(effects
@@
 			(project "LP5812_dev_board"
 				(path "/a5e340e1-6f5a-42cd-9c9f-a895aae72132"
-					(reference "TP?")
+					(reference "TP6")
 					(unit 1)
 				)
@@
 		(on_board yes)
 		(dnp yes)
-		(property "Reference" "TP?"
+		(property "Reference" "TP7"
 			(at 252.984 64.262 0)
 			(effects
@@
 			(project "LP5812_dev_board"
 				(path "/a5e340e1-6f5a-42cd-9c9f-a895aae72132"
-					(reference "TP?")
+					(reference "TP7")
 					(unit 1)
 				)
@@
 		(on_board yes)
 		(dnp yes)
-		(property "Reference" "TP?"
+		(property "Reference" "TP2"
 			(at 212.09 99.06 0)
 			(effects
@@
 			(project "LP5812_dev_board"
 				(path "/a5e340e1-6f5a-42cd-9c9f-a895aae72132"
-					(reference "TP?")
+					(reference "TP2")
 					(unit 1)
 				)
@@
 		(on_board yes)
 		(dnp yes)
-		(property "Reference" "TP?"
+		(property "Reference" "TP5"
 			(at 212.09 64.77 0)
 			(effects
@@
 			(project "LP5812_dev_board"
 				(path "/a5e340e1-6f5a-42cd-9c9f-a895aae72132"
-					(reference "TP?")
+					(reference "TP5")
 					(unit 1)
 				)
@@
 		(on_board yes)
 		(dnp yes)
-		(property "Reference" "TP?"
+		(property "Reference" "TP3"
 			(at 252.476 34.29 0)
 			(effects
@@
 			(project "LP5812_dev_board"
 				(path "/a5e340e1-6f5a-42cd-9c9f-a895aae72132"
-					(reference "TP?")
+					(reference "TP3")
 					(unit 1)
 				)
@@
 		(on_board yes)
 		(dnp yes)
-		(property "Reference" "TP?"
+		(property "Reference" "TP1"
 			(at 212.09 34.036 0)
 			(effects
@@
 			(project "LP5812_dev_board"
 				(path "/a5e340e1-6f5a-42cd-9c9f-a895aae72132"
-					(reference "TP?")
+					(reference "TP1")
 					(unit 1)
 				)

Commit message: Mark header as DNP
Parts:
- J1: now not fitted
Changed lines of the file:
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@@
 		(in_bom yes)
 		(on_board yes)
-		(dnp no)
+		(dnp yes)
 		(fields_autoplaced yes)
 		(property "Reference" "J1"
